File: 2040/hardware/kicad/PicoVerse2040.kicad_pcb (KiCad board)
At the start: 2 copper layers, 99.8 x 65 mm, 22 parts, among them Q1 BSS138, Q2 BSS138, Q3 BSS138, Q4 BSS138, Q5 BSS138, U1 WeAct-RP2040-Pico

Commit message: Fix pcb
Connections:
- C1 pad 1: /+5V -> GND
- C1 pad 2: GND -> /+5V
Changed lines of the file:
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@@
 			(layers "F.Cu" "F.Mask" "F.Paste")
 			(roundrect_rratio 0.25)
-			(net "/+5V")
+			(net "GND")
 			(pintype "passive")
 		)
@@
 			(layers "F.Cu" "F.Mask" "F.Paste")
 			(roundrect_rratio 0.25)
-			(net "GND")
+			(net "/+5V")
 			(pintype "passive")
 		)
@@
 	)
 	(segment
+		(start 160 97.175)
+		(end 160 94.2275)
+		(width 0.2)
+		(layer "F.Cu")
+		(net "/~{IORQ_33}")
+	)
+	(segment
+		(start 166.55 86.22)
+		(end 164.4487 88.3213)
+		(width 0.2)
+		(layer "F.Cu")
+		(net "/~{IORQ_33}")
+	)
+	(segment
+		(start 164.4487 88.3213)
+		(end 164.0387 88.3213)
+		(width 0.2)
+		(layer "F.Cu")
+		(net "/~{IORQ_33}")
+	)
+	(segment
+		(start 160.115 92.245)
+		(end 160.115 94.1125)
+		(width 0.2)
+		(layer "F.Cu")
+		(net "/~{IORQ_33}")
+	)
+	(segment
+		(start 160 94.2275)
+		(end 160.115 94.1125)
+		(width 0.2)
+		(layer "F.Cu")
+		(net "/~{IORQ_33}")
+	)
+	(segment
+		(start 164.0387 88.3213)
+		(end 160.115 92.245)
+		(width 0.2)
+		(layer "F.Cu")
+		(net "/~{IORQ_33}")
+	)
+	(segment
+		(start 159.99 97.185)
+		(end 160 97.175)
+		(width 0.2)
+		(layer "F.Cu")
+		(net "/~{IORQ_33}")
+	)
+	(segment
+		(start 166.55 84.23)
+		(end 166.55 86.22)
+		(width 0.2)
+		(layer "F.Cu")
+		(net "/~{IORQ_33}")
+	)
+	(via
+		(at 166.55 84.23)
+		(size 1.6)
+		(drill 1)
+		(layers "F.Cu" "B.Cu")
+		(capping no)
+		(covering
+			(front no)
+			(back no)
+		)
+		(plugging
+			(front no)
+			(back no)
+		)
+		(filling no)
+		(net "/~{IORQ_33}")
+	)
+	(segment
 		(start 170.23393 94.1125)
 		(end 169.855 94.1125)
@@
 	)
 	(segment
-		(start 160 97.175)
-		(end 160 94.2275)
-		(width 0.2)
-		(layer "F.Cu")
-		(net "/~{IORQ_33}")
-	)
-	(segment
-		(start 166.55 86.22)
-		(end 164.4487 88.3213)
-		(width 0.2)
-		(layer "F.Cu")
-		(net "/~{IORQ_33}")
-	)
-	(segment
-		(start 164.4487 88.3213)
-		(end 164.0387 88.3213)
-		(width 0.2)
-		(layer "F.Cu")
-		(net "/~{IORQ_33}")
-	)
-	(segment
-		(start 160.115 92.245)
-		(end 160.115 94.1125)
-		(width 0.2)
-		(layer "F.Cu")
-		(net "/~{IORQ_33}")
-	)
-	(segment
-		(start 160 94.2275)
-		(end 160.115 94.1125)
-		(width 0.2)
-		(layer "F.Cu")
-		(net "/~{IORQ_33}")
-	)
-	(segment
-		(start 164.0387 88.3213)
-		(end 160.115 92.245)
-		(width 0.2)
-		(layer "F.Cu")
-		(net "/~{IORQ_33}")
-	)
-	(segment
-		(start 159.99 97.185)
-		(end 160 97.175)
-		(width 0.2)
-		(layer "F.Cu")
-		(net "/~{IORQ_33}")
-	)
-	(segment
-		(start 166.55 84.23)
-		(end 166.55 86.22)
-		(width 0.2)
-		(layer "F.Cu")
-		(net "/~{IORQ_33}")
-	)
-	(via
-		(at 166.55 84.23)
-		(size 1.6)
-		(drill 1)
-		(layers "F.Cu" "B.Cu")
-		(capping no)
-		(covering
-			(front no)
-			(back no)
-		)
-		(plugging
-			(front no)
-			(back no)
-		)
-		(filling no)
-		(net "/~{IORQ_33}")
-	)
-	(segment
