File: 2040/hardware/kicad/PicoVerse2040-kp11.kicad_sch (KiCad schematic)
At the start: 25 parts, among them J1 MSX_Slot, Q1 BSS138, Q2 BSS138, Q3 BSS138, Q4 BSS138, Q5 BSS138, U1 WeAct-RP2040-Pico

Commit message: Working 7
Connections:
- net +5V: now also D4.16 (VCC), D5.16 (VCC)
- net GND: now also D4.15 (~{OE}), D4.8 (GND), D5.15 (~{OE}), D5.8 (GND)

Commit message: Make MUX_ADDR working
Parts:
- added U2: 74LVC1G32, symbol 74xGxx:74LVC1G32
Connections:
- net +5V: now also U2.5 (VCC)
- net ASEL: now also U2.4; no longer U1.1 (GP0)
- net GND: now also U2.3 (GND)
- net ~{IORQ_33}: no longer Q4.2 (S), R10.2
- net at U1.3 (GP2): now also U2.2
- net SLTSL renamed ~{SLTSL}
- new net: Q4.2 (S), R10.2
- new net: U1.1 (GP0), U2.1

Commit message: Add SD to MUX_ADDR
Parts:
- added J2: Micro_SD_Card, Connector_Card:microSD_HC_Wuerth_693072010801, symbol Connector:Micro_SD_Card
Connections:
- net GND: now also J2.6 (VSS), J2.9 (SHIELD)
- net MOSI: now reaches U1.4 (GP3)
- net MOSI: now also J2.3 (DI/MOSI)
- net MISO: now reaches U1.5 (GP4)
- net MISO: now also J2.7 (DO/MISO)
- net ~{SD_CS}: now reaches U1.7 (GP5)
- net ~{SD_CS}: now also J2.2 (nCS)
- net CLK: now reaches U1.8 (GP6)
- net CLK: now also J2.5 (CLK)
- new net +3V3: J2.4 (VDD)
